File: PCB_V01/MOUNTAIN_IN_THE_POCKET/MOUNTAIN_IN_THE_POCKET.kicad_sch (KiCad schematic)
At the start: 0 parts

Commit message: Actu kicad
Parts:
- added D1, D2, D3, D4: 14.2mm_157142S12703, Display7Segment_THT_Wurth:D_Wurth_WL-T7DS-14.2mm, symbol Display7Segment_Wurth_WL-T7DS:14.2mm_157142S12703
- added R1: NORPS-12, symbol Device:R_Photo
- added S1: SEN0137, symbol COMPONENTES_SCH:SEN0137
- added S2: SEN0251, symbol COMPONENTES_SCH:SEN0251
- added U1: AS1115-BSST, Package_SO:QSOP-24_3.9x8.7mm_P0.635mm, symbol Interface_Expansion:AS1115-BSST
- added VR1: 3362P-1-103LF, 3362P_1, symbol 3362P-1-103LF:3362P-1-103LF
Connections:
- new net: D3.3, D3.8
- new net: D2.3, D2.8
- new net: D4.3, D4.8
- new net: D1.3, D1.8
- new net +3V3: U1.19 (VDD)
- new net GND: U1.6 (GND)
- no-connect marks 0 -> 7
Other:
- note added: "potenciometro"

Commit message: SCH en proceso
Parts:
- removed S1: SEN0137, symbol COMPONENTES_SCH:SEN0137
- removed S2: SEN0251, symbol COMPONENTES_SCH:SEN0251
- added C1: C_Small, symbol Device:C_Small
- added D5, D6, D7: LED, symbol Device:LED
- added D9: M7, M7:DIOM505270X240, symbol M7:M7
- added J1: CON_ALIM, symbol Connector:Screw_Terminal_01x02
- added LS1: CEM-1205-IC, CEM1205IC, symbol CEM-1205-IC:CEM-1205-IC
- added Q1: 2N7002, SOT96P240X120-3N, symbol 2N7002:2N7002
- added R2, R3: 4k7, symbol Device:R_US
- added R4: 27k, symbol Device:R_US
- added R5: 100k, symbol Device:R_US
- added R6, R7, R8: R_US, symbol Device:R_US
- added R9: 220, symbol Device:R_US
- added S1: SEN0251, symbol COMPONENTES_SCH:SEN0251
- added S2: SEN0137, symbol COMPONENTES_SCH:SEN0137
- added SW1: SW_MEC_5E, symbol Switch:SW_MEC_5E
- added SW2: SWITCH_ALIM, Button_Switch_SMD:Nidec_Copal_CAS-120A, symbol Switch:SW_Nidec_CAS-120A1
- added UC1: (no value), ESP32_TOOLS_DIEGO:ESP32_WROOM32_SHIELD_V01, symbol ESP32_TOOLS_DIEGO:ESP32_WROOM32_SHIELD_V01
Connections:
- net +3V3: now also R1.1, R2.2, R3.1, R4.1
- net GND: now also VR1.3 (CW), C1.2, Q1.2 (S), R5.1, R6.1, R7.1, R8.1, S1.0 (GND), S2.0 (GND), SW1.1, SW1.2, UC1.14 (GND), UC1.20 (GND), UC1.26 (GND)
- net SEG_E: now reaches D3.1 (E)
- net SEG_E: now also D1.1 (E), D2.1 (E), D4.1 (E), U1.21 (SEGE)
- net SEG_G: now reaches D3.10 (G)
- net SEG_G: now also D1.10 (G), D2.10 (G), D4.10 (G), U1.18 (SEGG)
- net SEG_D: now reaches D3.2 (D)
- net SEG_D: now also D1.2 (D), D2.2 (D), D4.2 (D), U1.23 (SEGD)
- net DIG_3: now reaches D3.3, D3.8
- net DIG_3: now also U1.5 (DIG3)
- net SEG_C: now reaches D3.4 (C)
- net SEG_C: now also D1.4 (C), D2.4 (C), D4.4 (C), U1.20 (SEGC)
- net SEG_DP: now reaches D3.5 (DP)
- net SEG_DP: now also D1.5 (DP), D2.5 (DP), D4.5 (DP), U1.22 (SEGDP)
- net SEG_B: now reaches D3.6 (B)
- net SEG_B: now also D1.6 (B), D2.6 (B), D4.6 (B), U1.17 (SEGB)
- net SEG_A: now reaches D3.7 (A)
- net SEG_A: now also D1.7 (A), D2.7 (A), D4.7 (A), U1.15 (SEGA)
- net SEG_F: now reaches D3.9 (F)
- net SEG_F: now also D1.9 (F), D2.9 (F), D4.9 (F), U1.16 (SEGF)
- net DIG_1: now reaches D2.3, D2.8
- net DIG_1: now also U1.3 (DIG1)
- net DIG_2: now reaches D4.3, D4.8
- net DIG_2: now also U1.4 (DIG2)
- net at VR1.1 (CCW): now also R1.2
- net PIN_LDR: now reaches VR1.2 (WIPER)
- net DIG_0: now reaches D1.3, D1.8
- net DIG_0: now also U1.2 (DIG0)
- net SDA: now reaches U1.1 (SDA)
- net SDA: now also R3.2, S1.3 (SDA), UC1.25 (GPIO21)
- net at U1.13 (ISET): now also R4.2
- net SCL: now reaches U1.14 (SCL)
- net SCL: now also R2.1, S1.2 (SCL), UC1.22 (GPIO22)
- new net: D9.A, LS1., Q1.3 (D)
- new net: D5.1 (K), R6.2
- new net: D7.1 (K), R8.2
- new net: Q1.1 (G), R5.2, R9.1
- new net: D6.1 (K), R7.2
- new net +5V: D9.C, LS1.2, S2. (VCC), UC1.19 (5V)
- new net PIN_BUTTON: C1.1, SW1.3 (K), SW1.4 (A)
- new net PIN_BUZZER: R9.2
- new net PIN_SEN0137: S2.2 (DATA)
- no-connect marks 7 -> 9
Other:
- note added: "* REVISAR VCC"
- note added: "BARÓMETRO"
- note added: "BUZZER"
- note added: "C cerámico para filtrar alta f de conmutación?"
- note added: "Calcular resistencias y elegir colores de los diodos"
- note added: "DISPLAY 7 SEG"
- note added: "FUENTE DE ALIMENTACIÓN"
- note added: "GPIO con cuidado: 0, 2, 5, 12, 14, 15, 34, 35, 36, 39 Resto libres"
- note added: "LDR"
- note added: "LEDs"
- note added: "MICROCONTROLADOR"
- note added: "Poner switch para la alimentación, mejor antes de la fuente. Se podría poner otro extra a la salida de la fuente."
- note added: "Revisar que esté bien configurado ISET"
- note added: "SENSOR DE TEMPERATURA Y HUMEDAD"
- note added: "SENSORES E INPUTS"
- note added: "Saca 3V3 con 5V de alim"
- moved on the sheet: R1, U1

Commit message: buck
Parts:
- added C2: 10uF 50V, Capacitor_SMD:C_1206_3216Metric_Pad1.33x1.80mm_HandSolder, symbol Device:C
- added C3: 0.1uF 50V, Capacitor_SMD:C_0805_2012Metric_Pad1.18x1.45mm_HandSolder, symbol Device:C_Small
- added C4, C5: 22uF 10V, Capacitor_SMD:C_1206_3216Metric_Pad1.33x1.80mm_HandSolder, symbol Device:C
- added L1: 4.7uH 20%, Inductor_SMD:L_1008_2520Metric_Pad1.43x2.20mm_HandSolder, symbol Device:L
- added U2: AP63205WU, Package_TO_SOT_SMD:TSOT-23-6, symbol Regulator_Switching:AP63205WU
Connections:
- net +5V: now also C4.1, C5.1, L1.2, U2.1 (FB)
- net GND: now also C2.2, C4.2, C5.2, U2.4 (GND)
- new net: C3.2, L1.1, U2.5 (SW)
- new net: C3.1, U2.6 (BST)
- new net VBUS: C2.1, U2.2 (EN), U2.3 (IN)
Other:
- moved on the sheet: SW2

Commit message: Sesion 2 de octubre
Parts:
- removed C5: 22uF 10V, Capacitor_SMD:C_1206_3216Metric_Pad1.33x1.80mm_HandSolder, symbol Device:C
- removed D2, D3, D4: 14.2mm_157142S12703, Display7Segment_THT_Wurth:D_Wurth_WL-T7DS-14.2mm, symbol Display7Segment_Wurth_WL-T7DS:14.2mm_157142S12703
- removed SW2: SWITCH_ALIM, Button_Switch_SMD:Nidec_Copal_CAS-120A, symbol Switch:SW_Nidec_CAS-120A1
- added BT1: Battery, symbol Device:Battery
- added C10, C11, C3, C7: 0.1uF 50V, Capacitor_SMD:C_0805_2012Metric_Pad1.18x1.45mm_HandSolder, symbol Device:C_Small
- added C6: 22uF 10V, Capacitor_SMD:C_1206_3216Metric_Pad1.33x1.80mm_HandSolder, symbol Device:C
- added C9: 47uF 16V, CAPAE660X570N, symbol 865230343004:865230343004
- added D6, D7, D8: 14.2mm_157142S12703, Display7Segment_THT_Wurth:D_Wurth_WL-T7DS-14.2mm, symbol Display7Segment_Wurth_WL-T7DS:14.2mm_157142S12703
- added IC1: AZ1117CH-3.3TRG1, SOT230P700X180-4N, symbol AZ1117CH-3_3TRG1:AZ1117CH-3.3TRG1
- added JP1: SolderJumper_2_Open, symbol Jumper:SolderJumper_2_Open
- added JP2: Jumper_2_Open, symbol Jumper:Jumper_2_Open
- added Q3: (no value), Package_TO_SOT_SMD:TSOT-23_HandSoldering, symbol COMPONENTES_SCH:MMFTP3160
- added R2: 10k, Resistor_SMD:R_1206_3216Metric_Pad1.30x1.75mm_HandSolder, symbol Device:R_US
- added R8: 4k7, Resistor_SMD:R_1206_3216Metric_Pad1.30x1.75mm_HandSolder, symbol Device:R_US
- added S3: 1825232-1, 18252321, symbol 1825232-1:1825232-1
- C2: LINK (none) -> https://es.farnell.com/taiyo-yuden/umk325ab7106mm-t/condens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
- C4: renamed from C3; LINK (none) -> https://es.farnell.com/kyocera-avx/08055c104kat2a/conden-0-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
- C5: renamed from C4; LINK (none) -> https://es.farnell.com/semco/cl31b226mphnnne/cond-mlcc-22uf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
- D1: renamed from D5; value LED -> RED; footprint (none) -> LED_SMD:LED_1206_3216Metric_Pad1.42x1.75mm_HandSolder; LINK (none) -> https://es.farnell.com/lumex/sml-lx1206src-tr/led-red-2mm-x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
- D2: renamed from D6; value LED -> GREEN; footprint (none) -> LED_SMD:LED_1206_3216Metric_Pad1.42x1.75mm_HandSolder; LINK (none) -> https://es.farnell.com/lumex/sml-lxl1206gc-tr/led-green-1-1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
- D3: renamed from D7; value LED -> YELLOW; footprint (none) -> LED_SMD:LED_1206_3216Metric_Pad1.42x1.75mm_HandSolder; LINK (none) -> https://es.farnell.com/lumex/sml-lx1206syc-tr/led-amarillo-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
- D4: renamed from D9; LINK (none) -> https://es.farnell.com/multicomp-pro/1n4007-gs1g-m4/rectifi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
- D5: renamed from D1; LINK (none) -> https://es.farnell.com/wurth-elektronik/157142s12703/pantal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
- LS1: LINK (none) -> https://es.farnell.com/same-sky/cem-1205-ic/transudct-zumb-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
- Q1: LINK (none) -> https://es.farnell.com/onsemi/2n7002/mosfet-n-ch-60v-115ma-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
- R10: renamed from R9; footprint (none) -> Resistor_SMD:R_1206_3216Metric_Pad1.30x1.75mm_HandSolder; LINK (none) -> https://es.farnell.com/multicomp-pro/mcpwr06fteq2200a/res-2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
- R11: renamed from R5; value 100k -> 10k; footprint (none) -> Resistor_SMD:R_1206_3216Metric_Pad1.30x1.75mm_HandSolder; LINK (none) -> https://es.farnell.com/multicomp-pro/mcpwr06fteq1002a/res-1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
- R3: value 4k7 -> 100R; footprint (none) -> Resistor_SMD:R_1206_3216Metric_Pad1.30x1.75mm_HandSolder; LINK (none) -> https://es.farnell.com/bourns/crm1206-fx-1000elf/res-100r-1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
- R7: renamed from R2; footprint (none) -> Resistor_SMD:R_1206_3216Metric_Pad1.30x1.75mm_HandSolder; LINK (none) -> https://es.farnell.com/bourns/chp1206afx-4701elf/res-aec-q2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
- R9: renamed from R4; footprint (none) -> Resistor_SMD:R_1206_3216Metric_Pad1.30x1.75mm_HandSolder; LINK (none) -> https://es.farnell.com/vishay/crcw120625k5fkea/res-thick-fi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
- SW1: footprint (none) -> Button_Switch_SMD:SW_MEC_5GSH9; LINK (none) -> https://es.farnell.com/multicomp-pro/mptsm-21r-s-v/int-t-ct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
- U2: renamed from U1; LINK (none) -> https://es.farnell.com/ams-osram-group/as1115-bsst/display-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
- VR1: LINK (none) -> https://es.farnell.com/bourns/3362p-1-103lf/pot-trimmer-10k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
- renumbered R6 to R4, R7 to R5, R8 to R6, S2 to S1, S1 to S2, U2 to U1
Connections:
- net +3V3: now also D3.2 (A), S2.1 (VCC), C11.1, IC1.2 (OUTPUT), IC1.4 (VOUT), R8.2; no longer R3.1
- net +5V: now also D2.2 (A), C10.1, C6.1, C7.1, C9.1 (+), IC1.3 (INPUT)
- net DIG_1: now also D7.3, D7.8
- net DIG_2: now also D6.3, D6.8
- net DIG_3: now also D8.3, D8.8
- net GND: now also J1.1 (Pin_1), BT1.2 (-), C10.2, C11.2, C3.2, C6.2, C7.2, C9.2 (-), S3.3, S3.MH1, S3.MH2
- net SDA: now also R8.1; no longer R3.2
- net SEG_A: now also D6.7 (A), D7.7 (A), D8.7 (A)
- net SEG_B: now also D6.6 (B), D7.6 (B), D8.6 (B)
- net SEG_C: now also D6.4 (C), D7.4 (C), D8.4 (C)
- net SEG_D: now also D6.2 (D), D7.2 (D), D8.2 (D)
- net SEG_DP: now also D6.5 (DP), D7.5 (DP), D8.5 (DP)
- net SEG_E: now also D6.1 (E), D7.1 (E), D8.1 (E)
- net SEG_F: now also D6.9 (F), D7.9 (F), D8.9 (F)
- net SEG_G: now also D6.10 (G), D7.10 (G), D8.10 (G)
- net VBUS: now also D1.2 (A), J1.2 (Pin_2), JP1.1 (A), JP2.1 (A), Q3.2 (S), R2.2; no longer C2.1, U1.2 (EN), U1.3 (IN)
- new net: Q3.1 (G), R2.1, R3.1
- new net: R3.2, S3.2
- new net +BATT: BT1.1 (+), JP1.2 (B)
- new net VCC: C2.1, C3.1, JP2.2 (B), Q3.3 (D), U1.2 (EN), U1.3 (IN)
- no-connect marks 9 -> 10
Other:
- note removed: "* REVISAR VCC"
- note removed: "C cerámico para filtrar alta f de conmutación?"
- moved on the sheet: C1, C2, C4, C5, D1, D2, D3, D4, D5, L1, LS1, Q1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

Commit message: pcb actu
Parts:
- removed R4: R_US, symbol Device:R_US
- added C12: 22uF 10V, Capacitor_SMD:C_1206_3216Metric_Pad1.33x1.80mm_HandSolder, symbol Device:C
- added C13, C14, C15: 0.1uF 50V, Capacitor_SMD:C_0805_2012Metric_Pad1.18x1.45mm_HandSolder, symbol Device:C_Small
- added C8: 10 uF, Capacitor_SMD:C_1206_3216Metric_Pad1.33x1.80mm_HandSolder, symbol Device:C
- added R12: 10k, Resistor_SMD:R_1206_3216Metric_Pad1.30x1.75mm_HandSolder, symbol Device:R_US
- R10: value 220 -> 220R
- R5: value R_US -> 3k; footprint (none) -> Resistor_SMD:R_1206_3216Metric_Pad1.30x1.75mm_HandSolder; LINK (none) -> https://es.farnell.com/yageo/rc1206fr-073kl/resis-3k-1-0-25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
- R6: value R_US -> 1K3; footprint (none) -> Resistor_SMD:R_1206_3216Metric_Pad1.30x1.75mm_HandSolder; LINK (none) -> https://es.farnell.com/panasonic/erj8geyj132v/res-1k3-5-0-2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
- S1: footprint (none) -> LIB_HUELLAS_MITP:CONECTOR_0137
- S2: footprint (none) -> LIB_HUELLAS_MITP:CONECTOR_0251
Connections:
- net +3V3: now also C12.1, C14.1, C15.2
- net +5V: now also S1.1 (VCC), C13.1, C8.1; no longer S1. (VCC)
- net GND: now also IC1.1 (ADJ/GND), C12.2, C13.2, C14.2, C15.1, C8.2, R12.1
- net PIN_BUTTON: now also UC1.30 (GPIO17)
- net PIN_BUZZER: now also UC1.15 (GPIO13)
- net PIN_LDR: now also UC1.8 (GPIO33)
- net PIN_SEN0137: now also UC1.32 (GPIO04)
- net at D1.1 (K): now also R12.2
Other:
- note removed: "Saca 3V3 con 5V de alim"
- moved on the sheet: BT1, C1, C10, C11, C2, C3, C4, C5, C6, C7, C9, D1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

Commit message: update footprints
Parts:
- added C16: C_Small, symbol Device:C_Small
- added SW2: SW_MEC_5E, Button_Switch_SMD:SW_MEC_5GSH9, symbol Switch:SW_MEC_5E
Connections:
- net GND: now also C16.2, SW2.1, SW2.2
- net PIN_BUTTON_2: now reaches UC1.31 (GPIO16)
- net PIN_BUTTON_2: now also C16.1, SW2.3 (K), SW2.4 (A)
- net PIN_BUTTON renamed PIN_BUTTON_1

Commit message: Actualizaciones con footprints
Parts:
- removed C1, C16: C_Small, symbol Device:C_Small
- added C4, C5: 0.1uF 50V, Capacitor_SMD:C_0805_2012Metric_Pad1.18x1.45mm_HandSolder, symbol Device:C_Small
- added R1, R3: 10k, Resistor_SMD:R_1206_3216Metric_Pad1.30x1.75mm_HandSolder, symbol Device:R_US
- C8: renamed from C9; footprint CAPAE660X570N -> CAPAE660X570N:CAPAE660X570N
- D4: footprint M7:DIOM505270X240 -> Diode_SMD:D_SMA_Handsoldering
- SW1, SW2: footprint Button_Switch_SMD:SW_MEC_5GSH9 -> TL3305AF160QG:TL3305AF160QG; LINK https://es.farnell.com/multicomp-pro/mptsm-21r-s-v/int-t-ct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 -> https://es.farnell.com/e-switch/tl3305af160qg/int-t-ctil-0-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
- renumbered C15 to C1, C4 to C10, C5 to C11, C6 to C12, C8 to C13, C11 to C14, C12 to C15, C10 to C16, C13 to C2, C14 to C3, C2 to C6, C3 to C7, C7 to C9, Q3 to Q1, Q1 to Q2, R8 to R10, R9 to R11, R10 to R12, R11 to R13, R1 to R2, R2 to R4, R3 to R5, R12 to R6, R5 to R7, R6 to R8, R7 to R9
Connections:
- net +5V: now also D4.1 (C); no longer D4.C
- net GND: now also C4.2, C5.2, R1.1, R3.1; no longer SW1.1, SW1.2, SW2.1, SW2.2
- net PIN_BUTTON_1: now also C4.1
- net PIN_BUTTON_2: now also C5.1
- new net: D4.2 (A), LS1.1, Q2.3 (D)
- new net: R1.2, SW1.1, SW1.2
- new net: R3.2, SW2.1, SW2.2

Commit message: Esquemático v1.0 terminado
Parts:
- removed BT1: Battery, symbol Device:Battery
- removed D4: M7, Diode_SMD:D_SMA_Handsoldering, symbol M7:M7
- removed JP1: SolderJumper_2_Open, symbol Jumper:SolderJumper_2_Open
- added CX17, CX18: C, Capacitor_THT:C_Rect_L41.5mm_W40.0mm_P37.50mm_MKS4, symbol Device:C
- added D4: D, Diode_SMD:D_SMA_Handsoldering, symbol Device:D
- added JP3: Jumper_2_Open, Connector_PinHeader_2.54mm:PinHeader_2x01_P2.54mm_Vertical, symbol Jumper:Jumper_2_Open
- added JP4, JP5: Jumper_2_Small_Open, Connector_PinHeader_2.54mm:PinHeader_2x01_P2.54mm_Vertical, symbol Jumper:Jumper_2_Small_Open
- added L2: L_Ferrite_Coupled_1243, Inductor_THT:Choke_EPCOS_B82722A, symbol Device:L_Ferrite_Coupled_1243
- J1: footprint (none) -> TerminalBlock_Phoenix:TerminalBlock_Phoenix_MKDS-1,5-2-5.08_1x02_P5.08mm_Horizontal; Link (none) -> https://es.farnell.com/phoenix-contact/1729128/bloque-termi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
- JP2: footprint (none) -> Connector_PinHeader_2.54mm:PinHeader_2x01_P2.54mm_Vertical
- R2: footprint (none) -> LIB_HUELLAS_MITP:NORPS12
Connections:
- net +5V: now also D4.1 (K)
- net GND: now also JP5.1 (A), L2.3; no longer J1.1 (Pin_1)
- net VBUS: now also CX17.1, JP3.2 (B), L2.2; no longer J1.2 (Pin_2)
- net at LS1.1, Q2.3 (D): now also D4.2 (A)
- new net: CX17.2, JP5.2 (B)
- new net: CX18.1, J1.2 (Pin_2), JP3.1 (A), L2.1
- new net: J1.1 (Pin_1), JP4.1 (A), L2.4
- new net: CX18.2, JP4.2 (B)
Other:
- note added: "IDEA"
- note added: "PONER FUSIBLE"
- note added: "Poner jumpers en las alimentaciones de las cosas para ver de donde viene el ruido"
- note added: "Recordar que en el BOM tiene que estar la parte de arriba de los jumpers"
- moved on the sheet: C10, C11, C12, C13, C15, C6, C7, C8, C9, IC1, J1, JP2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
