File: PCB_V01/MOUNTAIN_IN_THE_POCKET/MOUNTAIN_IN_THE_POCKET.kicad_sch (KiCad schematic)
At the start: 59 parts, among them IC1 AZ1117CH-3.3TRG1, J1 CON_ALIM, Q2 2N7002, SW1 SW_MEC_5E, SW2 SW_MEC_5E, U1 AP63205WU, U2 AS1115-BSST

Commit message: esquemático v1.1 y placement 1.0
Parts:
- added D9: RED, LED_SMD:LED_1206_3216Metric_Pad1.42x1.75mm_HandSolder, symbol Device:LED
- added R14: 10k, Resistor_SMD:R_1206_3216Metric_Pad1.30x1.75mm_HandSolder, symbol Device:R_US
- added R15: (no value), Resistor_SMD:R_1206_3216Metric_Pad1.30x1.75mm_HandSolder, symbol Device:R_US
- C8: now not fitted; now left out of the parts list
- Q2: footprint SOT96P240X120-3N -> Package_TO_SOT_SMD:SOT-23_Handsoldering
- R10, R9: now not fitted
Connections:
- net GND: now also R14.1, R15.1; no longer VR1.3 (CW)
- net VCC: now also D9.2 (A)
- new net: R15.2, VR1.3 (CW)
- new net: D9.1 (K), R14.2
Other:
- moved on the sheet: D1, R6

Commit message: routing de los visualizadores y placement
Connections:
- net PIN_LDR: now also R15.2, R2.2; no longer VR1.2 (WIPER)
- net at VR1.1 (CCW): no longer R2.2
- net at VR1.3 (CW): no longer R15.2
Other:
- moved on the sheet: C3, S2

Commit message: actualizado routing
Parts:
- added H1, H2, H3, H4: MountingHole, MountingHole:MountingHole_3.2mm_M3, symbol Mechanical:MountingHole

Commit message: actu routing
Parts:
- removed VR1: 3362P-1-103LF, 3362P_1, symbol 3362P-1-103LF:3362P-1-103LF
- added TP1: TEST_VBUS, TestPoint:TestPoint_THTPad_D1.0mm_Drill0.5mm, symbol Connector:TestPoint
- added TP2: TEST_VCC, TestPoint:TestPoint_THTPad_D1.0mm_Drill0.5mm, symbol Connector:TestPoint
- added TP3: TEST_5V, TestPoint:TestPoint_THTPad_D1.0mm_Drill0.5mm, symbol Connector:TestPoint
- added TP4: TEST_3V3, TestPoint:TestPoint_THTPad_D1.0mm_Drill0.5mm, symbol Connector:TestPoint
- added TP5: TEST_GND, TestPoint:TestPoint_THTPad_D1.0mm_Drill0.5mm, symbol Connector:TestPoint
- added TP6: TEST_SDA, TestPoint:TestPoint_THTPad_D1.0mm_Drill0.5mm, symbol Connector:TestPoint
- added TP7: TEST_SCL, TestPoint:TestPoint_THTPad_D1.0mm_Drill0.5mm, symbol Connector:TestPoint
- R2: footprint LIB_HUELLAS_MITP:NORPS12 -> OptoDevice:R_LDR_5.1x4.3mm_P3.4mm_Vertical; LINK https://es.farnell.com/advanced-photonix/norps-12/light-dep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 -> (none)
Connections:
- net +3V3: now also UC1.1 (3V3), TP4.1
- net +5V: now also TP3.1
- net GND: now also TP5.1
- net PIN_BUTTON_1: now also UC1.27 (GPIO19); no longer UC1.30 (GPIO17)
- net PIN_BUTTON_2: now also UC1.28 (GPIO18); no longer UC1.31 (GPIO16)
- net PIN_BUZZER: now also UC1.30 (GPIO17); no longer UC1.15 (GPIO13)
- net PIN_SEN0137: now also UC1.21 (GPIO23); no longer UC1.32 (GPIO04)
- net SCL: now also S2.3 (SCL), TP7.1; no longer S2.2 (SCL)
- net SDA: now also S2.2 (SDA), TP6.1; no longer S2.3 (SDA)
- net VBUS: now also TP1.1
- net VCC: now also TP2.1
- no-connect marks 10 -> 28
Other:
- moved on the sheet: C8, C9, D1, D2, D3, D9, R14, R6, R7, R8
