File: PCB_V01/MOUNTAIN_IN_THE_POCKET/MOUNTAIN_IN_THE_POCKET.kicad_pcb (KiCad board)
At the start: 2 copper layers, 1 part, among them U1 AS1115-BSST

Commit message: SCH en proceso
Parts:
- moved U1 21.8 mm to (33.1, 33.0)
Changed lines of the file:
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@@
 	(footprint "Package_SO:QSOP-24_3.9x8.7mm_P0.635mm"
 		(layer "F.Cu")
-		(at 53.925 39.625)
+		(at 33.125 33.025)
 		(descr "QSOP, 24 Pin (https://pdfserv.maximintegrated.com/package_dwgs/21-0055.PDF)")
 		(tags "QSOP SO")

Commit message: Sesion 2 de octubre
Parts:
- added C10: 0.1uF 50V, Capacitor_SMD:C_0805_2012Metric_Pad1.18x1.45mm_HandSolder, F.Cu at (54.3, 128.0)
- added C11: 0.1uF 50V, Capacitor_SMD:C_0805_2012Metric_Pad1.18x1.45mm_HandSolder, F.Cu at (54.3, 131.0)
- added C2: 10uF 50V, Capacitor_SMD:C_1206_3216Metric_Pad1.33x1.80mm_HandSolder, F.Cu at (27.4, 127.4)
- added C3: 0.1uF 50V, Capacitor_SMD:C_0805_2012Metric_Pad1.18x1.45mm_HandSolder, F.Cu at (26.8, 144.3)
- added C4: 0.1uF 50V, Capacitor_SMD:C_0805_2012Metric_Pad1.18x1.45mm_HandSolder, F.Cu at (26.8, 147.3)
- added C5: 22uF 10V, Capacitor_SMD:C_1206_3216Metric_Pad1.33x1.80mm_HandSolder, F.Cu at (27.4, 130.8)
- added C6: 22uF 10V, Capacitor_SMD:C_1206_3216Metric_Pad1.33x1.80mm_HandSolder, F.Cu at (27.4, 134.1)
- added C6: 22uF 10V, Capacitor_SMD:C_1206_3216Metric_Pad1.33x1.80mm_HandSolder, F.Cu at (59.7, 129.8)
- added C7: 0.1uF 50V, Capacitor_SMD:C_0805_2012Metric_Pad1.18x1.45mm_HandSolder, F.Cu at (54.3, 125.0)
- added D1: RED, LED_SMD:LED_1206_3216Metric_Pad1.42x1.75mm_HandSolder, F.Cu at (26.5, 171.2)
- added D2: GREEN, LED_SMD:LED_1206_3216Metric_Pad1.42x1.75mm_HandSolder, F.Cu at (26.5, 174.6)
- added D3: YELLOW, LED_SMD:LED_1206_3216Metric_Pad1.42x1.75mm_HandSolder, F.Cu at (26.5, 178.0)
- added L1: 4.7uH 20%, Inductor_SMD:L_1008_2520Metric_Pad1.43x2.20mm_HandSolder, F.Cu at (27.1, 150.7)
- added Q2: PMOS, Package_TO_SOT_SMD:TSOT-23_HandSoldering, F.Cu at (52.7, 172.8)
- added Q3: ~, Package_TO_SOT_SMD:TSOT-23_HandSoldering, F.Cu at (60.2, 125.9)
- added R10: 220, Resistor_SMD:R_1206_3216Metric_Pad1.30x1.75mm_HandSolder, F.Cu at (27.4, 117.5)
- added R11: 10k, Resistor_SMD:R_1206_3216Metric_Pad1.30x1.75mm_HandSolder, F.Cu at (27.4, 120.8)
- added R2: 10k, Resistor_SMD:R_1206_3216Metric_Pad1.30x1.75mm_HandSolder, F.Cu at (26.5, 181.3)
- added R3: 100R, Resistor_SMD:R_1206_3216Metric_Pad1.30x1.75mm_HandSolder, F.Cu at (26.5, 184.6)
- added R7: 4k7, Resistor_SMD:R_1206_3216Metric_Pad1.30x1.75mm_HandSolder, F.Cu at (27.4, 110.9)
- added R8: 4k7, Resistor_SMD:R_1206_3216Metric_Pad1.30x1.75mm_HandSolder, F.Cu at (27.4, 124.1)
- added R9: 27k, Resistor_SMD:R_1206_3216Metric_Pad1.30x1.75mm_HandSolder, F.Cu at (27.4, 114.2)
- added SW1: SWITCH_ALIM, Button_Switch_SMD:Nidec_Copal_CAS-120A, F.Cu at (27.1, 139.3)
- added U1: AP63205WU, Package_TO_SOT_SMD:TSOT-23-6, F.Cu at (27.0, 154.9)
- added UC1: ~, ESP32_TOOLS_DIEGO:ESP32_WROOM32_SHIELD_V01, F.Cu at (35.0, 98.7)
- renumbered U1 to U2
Connections:
- U2 pad 1: unconnected-(U1-SDA-Pad1) -> /SDA
- U2 pad 13: unconnected-(U1-ISET-Pad13) -> Net-(U2-ISET)
- U2 pad 14: unconnected-(U1-SCL-Pad14) -> /SCL
- U2 pad 15: unconnected-(U1-SEGA-Pad15) -> /SEG_A
- U2 pad 16: unconnected-(U1-SEGF-Pad16) -> /SEG_F
- U2 pad 17: unconnected-(U1-SEGB-Pad17) -> /SEG_B
- U2 pad 18: unconnected-(U1-SEGG-Pad18) -> /SEG_G
- U2 pad 2: unconnected-(U1-DIG0-Pad2) -> /DIG_0
- U2 pad 20: unconnected-(U1-SEGC-Pad20) -> /SEG_C
- U2 pad 21: unconnected-(U1-SEGE-Pad21) -> /SEG_E
- U2 pad 22: unconnected-(U1-SEGDP-Pad22) -> /SEG_DP
- U2 pad 23: unconnected-(U1-SEGD-Pad23) -> /SEG_D
- U2 pad 3: unconnected-(U1-DIG1-Pad3) -> /DIG_1
- U2 pad 4: unconnected-(U1-DIG2-Pad4) -> /DIG_2
- U2 pad 5: unconnected-(U1-DIG3-Pad5) -> /DIG_3

Commit message: update footprints
Parts:
- added C12: 22uF 10V, Capacitor_SMD:C_1206_3216Metric_Pad1.33x1.80mm_HandSolder, F.Cu at (-68.4, 38.5)
- added C13: 0.1uF 50V, Capacitor_SMD:C_0805_2012Metric_Pad1.18x1.45mm_HandSolder, F.Cu at (-57.3, 18.3)
- added C14: 0.1uF 50V, Capacitor_SMD:C_0805_2012Metric_Pad1.18x1.45mm_HandSolder, F.Cu at (-57.3, 21.4)
- added C15: 0.1uF 50V, Capacitor_SMD:C_0805_2012Metric_Pad1.18x1.45mm_HandSolder, F.Cu at (-57.3, 24.4)
- added C8: 10 uF, Capacitor_SMD:C_1206_3216Metric_Pad1.33x1.80mm_HandSolder, F.Cu at (-68.4, 35.2)
- added D5: 14.2mm_157142S12703, Display7Segment_THT_Wurth:D_Wurth_WL-T7DS-14.2mm, F.Cu at (28.8, 9.20)
- added D6: 14.2mm_157142S12703, Display7Segment_THT_Wurth:D_Wurth_WL-T7DS-14.2mm, F.Cu at (28.8, 23.3)
- added D7: 14.2mm_157142S12703, Display7Segment_THT_Wurth:D_Wurth_WL-T7DS-14.2mm, F.Cu at (28.8, 37.5)
- added D8: 14.2mm_157142S12703, Display7Segment_THT_Wurth:D_Wurth_WL-T7DS-14.2mm, F.Cu at (28.8, 51.6)
- added R12: 10k, Resistor_SMD:R_1206_3216Metric_Pad1.30x1.75mm_HandSolder, F.Cu at (-62.4, 41.8)
- added R5: 3k, Resistor_SMD:R_1206_3216Metric_Pad1.30x1.75mm_HandSolder, F.Cu at (-62.4, 35.1)
- added R6: 1K3, Resistor_SMD:R_1206_3216Metric_Pad1.30x1.75mm_HandSolder, F.Cu at (-62.4, 38.5)
- added S1: SEN0137, LIB_HUELLAS_MITP:CONECTOR_0137, F.Cu at (-81.1, 30.8)
- added S2: SEN0251, LIB_HUELLAS_MITP:CONECTOR_0251, F.Cu at (-78.4, 46.3)
- added SW1: SW_MEC_5E, Button_Switch_SMD:SW_MEC_5GSH9, F.Cu at (-65.6, 25.2)
- R10: value 220 -> 220R
- moved C11 45.6 mm to (10.3, 119.4)
- moved C2 45.6 mm to (-16.6, 115.8)
- moved C5 45.6 mm to (-16.6, 119.1)
- moved C6 45.6 mm to (15.7, 118.2)
- moved C7 45.6 mm to (10.3, 113.3)
- moved D1 45.6 mm to (-17.5, 159.5)
- moved D2 45.6 mm to (-17.5, 162.9)
- moved D3 45.6 mm to (-17.5, 166.3)
- moved Q2 45.6 mm to (8.67, 161.1)
- moved Q3 45.6 mm to (16.2, 114.3)
- moved R2 45.6 mm to (-17.6, 169.7)
- moved R3 45.6 mm to (-17.6, 173.0)
- moved U1 45.6 mm to (-17.0, 143.3)
- moved U2 45.6 mm to (-10.9, 21.4)
- moved UC1 45.6 mm to (-9.09, 87.0)
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Connections:
- UC1 pad 15: unconnected-(UC1-GPIO13-Pad15) -> /PIN_BUZZER
- UC1 pad 30: unconnected-(UC1-GPIO17-Pad30) -> /PIN_BUTTON
- UC1 pad 32: unconnected-(UC1-GPIO04-Pad32) -> /PIN_SEN0137
- UC1 pad 8: unconnected-(UC1-GPIO33-Pad8) -> /PIN_LDR

Commit message: Actualizaciones con footprints
Parts:
- removed the C6 at (-16.6, 122.5)
- removed the C6 at (15.7, 118.2)
- removed Q3: ~, Package_TO_SOT_SMD:TSOT-23_HandSoldering
- removed R2: 10k, Resistor_SMD:R_1206_3216Metric_Pad1.30x1.75mm_HandSolder
- removed the SW1 at (-16.9, 127.6)
- removed the SW1 at (-65.6, 25.2)
- added C1: 0.1uF 50V, Capacitor_SMD:C_0805_2012Metric_Pad1.18x1.45mm_HandSolder, F.Cu at (-19.4, 60.9)
- added C16: 0.1uF 50V, Capacitor_SMD:C_0805_2012Metric_Pad1.18x1.45mm_HandSolder, F.Cu at (-14.6, 73.0)
- added C6: 10uF 50V, Capacitor_SMD:C_1206_3216Metric_Pad1.33x1.80mm_HandSolder, F.Cu at (-9.21, 61.1)
- added C9: 0.1uF 50V, Capacitor_SMD:C_0805_2012Metric_Pad1.18x1.45mm_HandSolder, F.Cu at (-14.6, 63.9)
- added D4: M7, Diode_SMD:D_SMA_Handsoldering, F.Cu at (-66.0, 81.1)
- added IC1: AZ1117CH-3.3TRG1, AZ1117CH-3.3TRG1:SOT230P700X180-4N, F.Cu at (-7.41, 80.3)
- added LS1: CEM-1205-IC, CEM-1205-IC:CEM1205IC, F.Cu at (-14.3, 17.9)
- added Q1: ~, Package_TO_SOT_SMD:TSOT-23_HandSoldering, F.Cu at (-4.99, 41.8)
- added R1: 10k, Resistor_SMD:R_1206_3216Metric_Pad1.30x1.75mm_HandSolder, F.Cu at (-39.5, 72.4)
- added R13: 10k, Resistor_SMD:R_1206_3216Metric_Pad1.30x1.75mm_HandSolder, F.Cu at (-27.6, 82.3)
- added R4: 10k, Resistor_SMD:R_1206_3216Metric_Pad1.30x1.75mm_HandSolder, F.Cu at (-39.5, 79.0)
- added S3: 1825232-1, 1825232-1:18252321, F.Cu at (-56.1, 71.1)
- added SW1: SW_MEC_5E, TL3305AF160QG:TL3305AF160QG, F.Cu at (-65.3, 70.2)
- added SW2: SW_MEC_5E, TL3305AF160QG:TL3305AF160QG, F.Cu at (-65.3, 76.0)
- added VR1: 3362P-1-103LF, 3362P-1-103LF-pretty:3362P_1, F.Cu at (-4.09, 52.3)
- C11, C15: value 0.1uF 50V -> 22uF 10V; footprint Capacitor_SMD:C_0805_2012Metric_Pad1.18x1.45mm_HandSolder -> Capacitor_SMD:C_1206_3216Metric_Pad1.33x1.80mm_HandSolder
- C13: value 0.1uF 50V -> 10 uF; footprint Capacitor_SMD:C_0805_2012Metric_Pad1.18x1.45mm_HandSolder -> Capacitor_SMD:C_1206_3216Metric_Pad1.33x1.80mm_HandSolder
- C2: value 10uF 50V -> 0.1uF 50V; footprint Capacitor_SMD:C_1206_3216Metric_Pad1.33x1.80mm_HandSolder -> Capacitor_SMD:C_0805_2012Metric_Pad1.18x1.45mm_HandSolder
- C5: value 22uF 10V -> 0.1uF 50V; footprint Capacitor_SMD:C_1206_3216Metric_Pad1.33x1.80mm_HandSolder -> Capacitor_SMD:C_0805_2012Metric_Pad1.18x1.45mm_HandSolder
- C8: value 10 uF -> 47uF 16V; footprint Capacitor_SMD:C_1206_3216Metric_Pad1.33x1.80mm_HandSolder -> CAPAE660X570N:CAPAE660X570N
- Q2: value PMOS -> 2N7002; footprint Package_TO_SOT_SMD:TSOT-23_HandSoldering -> 2N7002:SOT96P240X120-3N
- R10: value 220R -> 4k7
- R11: value 10k -> 27k
- R12: value 10k -> 220R
- R3: value 100R -> 10k
- R5: value 3k -> 100R
- R6: value 1K3 -> 10k
- R7: value 4k7 -> 3k
- R8: value 4k7 -> 1K3
- R9: value 27k -> 4k7
- moved D2 129.2 mm to (-5.45, 34.3)
- moved D1 129.2 mm to (-5.45, 30.9)
- moved D3 129.2 mm to (-5.45, 37.7)
- moved R3 99.8 mm to (-39.5, 75.7)
- moved Q2 97.0 mm to (-47.0, 81.7)
- moved L1 84.8 mm to (-5.82, 54.9)
- moved U1 72.5 mm to (-46.9, 77.2)
- moved C13 71.4 mm to (-9.21, 71.1)
- moved C15 69.5 mm to (-9.21, 74.5)
- moved D5 68.9 mm to (-39.7, 16.3)
- moved D6 68.9 mm to (-39.7, 30.4)
- moved D7 68.9 mm to (-39.7, 44.6)
- moved D8 68.9 mm to (-39.7, 58.7)
- moved S1 68.8 mm to (-18.1, 58.7)
- moved C12 66.0 mm to (-9.21, 67.8)
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Connections:
- C10 pad 1: +5V -> Net-(U1-BST)
- C10 pad 2: GND -> Net-(U1-SW)
- C11 pad 1: +3V3 -> +5V
- C12 pad 1: +3V3 -> +5V
- C15 pad 1: GND -> +3V3
- C15 pad 2: +3V3 -> GND
- C2 pad 1: VCC -> +5V
- C3 pad 1: VCC -> +3V3
- C4 pad 1: Net-(U1-BST) -> /PIN_BUTTON_1
- C4 pad 2: Net-(U1-SW) -> GND
- C5 pad 1: +5V -> /PIN_BUTTON_2
- C7 pad 1: +5V -> VCC
- Q2 pad 1: unconnected-(Q2-D-Pad1) -> Net-(Q2-G)
- Q2 pad 2: unconnected-(Q2-G-Pad2) -> GND
- Q2 pad 3: unconnected-(Q2-S-Pad3) -> Net-(D4-A)
- R10 pad 1: Net-(Q1-G) -> /SDA
- R10 pad 2: /PIN_BUZZER -> +3V3
- R11 pad 1: GND -> +3V3
- R11 pad 2: Net-(Q1-G) -> Net-(U2-ISET)
- R12 pad 1: GND -> Net-(Q2-G)
- R12 pad 2: Net-(D1-K) -> /PIN_BUZZER
- R3 pad 1: Net-(Q3-G) -> GND
- R5 pad 1: GND -> Net-(Q1-G)
- R5 pad 2: Net-(D2-K) -> Net-(R5-Pad2)
- R6 pad 2: Net-(D3-K) -> Net-(D1-K)
- R7 pad 1: /SCL -> GND
- R7 pad 2: +3V3 -> Net-(D2-K)
- R8 pad 1: /SDA -> GND
- R8 pad 2: +3V3 -> Net-(D3-K)
- R9 pad 1: +3V3 -> /SCL
- R9 pad 2: Net-(U2-ISET) -> +3V3
- UC1 pad 30: /PIN_BUTTON -> /PIN_BUTTON_1
- UC1 pad 31: unconnected-(UC1-GPIO16-Pad31) -> /PIN_BUTTON_2

Commit message: Esquemático v1.0 terminado
Parts:
- removed UC1: ~, ESP32_TOOLS_DIEGO:ESP32_WROOM32_SHIELD_V01
- added CX17: C, Capacitor_THT:C_Rect_L41.5mm_W40.0mm_P37.50mm_MKS4, F.Cu at (34.3, 101.8)
- added CX18: C, Capacitor_THT:C_Rect_L41.5mm_W40.0mm_P37.50mm_MKS4, F.Cu at (34.3, 143.3)
- added J1: CON_ALIM, TerminalBlock_Phoenix:TerminalBlock_Phoenix_MKDS-1,5-2-5.08_1x02_P5.08mm_Horizontal, F.Cu at (110.0, 158.6)
- added JP2: Jumper_2_Open, Connector_PinHeader_2.54mm:PinHeader_2x01_P2.54mm_Vertical, F.Cu at (91.9, 154.6)
- added JP3: Jumper_2_Open, Connector_PinHeader_2.54mm:PinHeader_2x01_P2.54mm_Vertical, F.Cu at (91.9, 159.2)
- added JP4: Jumper_2_Small_Open, Connector_PinHeader_2.54mm:PinHeader_2x01_P2.54mm_Vertical, F.Cu at (91.9, 163.8)
- added JP5: Jumper_2_Small_Open, Connector_PinHeader_2.54mm:PinHeader_2x01_P2.54mm_Vertical, F.Cu at (91.9, 168.4)
- added L2: L_Ferrite_Coupled_1243, Inductor_THT:Choke_EPCOS_B82722A, F.Cu at (41.0, 74.5)
- added R2: NORPS-12, LIB_HUELLAS_MITP:NORPS12, F.Cu at (99.2, 114.2)
- D4: value M7 -> D
- moved S3 193.0 mm to (110.7, 168.2)
- moved SW1 187.7 mm to (108.8, 140.4)
- moved SW2 187.7 mm to (108.8, 146.2)
- moved Q1 165.7 mm to (100.3, 169.8)
- moved D2 163.3 mm to (116.7, 142.7)
- moved D1 163.3 mm to (116.7, 139.3)
- moved D3 163.3 mm to (116.7, 146.1)
- moved Q2 156.7 mm to (82.1, 170.5)
- moved D4 156.7 mm to (65.4, 166.4)
- moved LS1 156.7 mm to (82.1, 141.3)
- moved S2 156.7 mm to (80.9, 167.4)
- moved U1 155.2 mm to (77.1, 170.6)
- moved C1 150.7 mm to (99.2, 153.8)
- moved C10 150.7 mm to (104.0, 159.9)
- moved C14 150.7 mm to (104.0, 162.9)
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
Commit message: LIBRERIA ESP
Parts:
- added UC1: ~, ESP32_TOOLS_DIEGO:ESP32_WROOM32_SHIELD_V01, F.Cu at (154.3, 122.0)

Commit message: esquemático v1.1 y placement 1.0
Parts:
- removed C8: 47uF 16V, CAPAE660X570N:CAPAE660X570N
- added D9: RED, LED_SMD:LED_1206_3216Metric_Pad1.42x1.75mm_HandSolder, F.Cu at (73.8, 90.5)
- added R14: 10k, Resistor_SMD:R_1206_3216Metric_Pad1.30x1.75mm_HandSolder, F.Cu at (77.8, 91.5)
- added R15: 10k, Resistor_SMD:R_1206_3216Metric_Pad1.30x1.75mm_HandSolder, F.Cu at (123.3, 57.3)
- Q2: footprint 2N7002:SOT96P240X120-3N -> Package_TO_SOT_SMD:SOT-23_Handsoldering
- moved D4 147.9 mm to (143.5, 40.8), turned to 90 degrees
- moved Q2 142.2 mm to (138.0, 39.8), turned to 90 degrees
- moved S2 136.0 mm to (131.7, 41.3), turned to 90 degrees
- moved CX17 132.3 mm to (-93.5, 67.5)
- moved CX18 132.3 mm to (-93.5, 109.0)
- moved L2 132.3 mm to (-86.8, 40.2)
- moved VR1 129.7 mm to (126.0, 62.3), turned to 90 degrees
- moved J1 127.8 mm to (69.0, 37.5), turned to 180 degrees
- moved C16 124.8 mm to (143.5, 47.5), turned to -90 degrees
- moved LS1 124.7 mm to (152.5, 38.5)
- moved IC1 122.0 mm to (135.5, 84.0), turned to -90 degrees
- moved C3 119.8 mm to (130.1, 44.1), turned to 90 degrees
- moved D1 110.3 mm to (77.2, 36.2), turned to 90 degrees
- moved JP3 106.9 mm to (65.2, 55.8)
- moved JP4 106.9 mm to (65.2, 60.3)
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Connections:
- VR1 pad 3: GND -> Net-(VR1-CW)

Commit message: routing de los visualizadores y placement
Parts:
- R15: value 10k -> ~
- moved LS1 53.0 mm to (130.0, 86.4), turned to -90 degrees
- moved C15 43.7 mm to (101.5, 103.5), turned to 180 degrees
- moved D4 39.7 mm to (127.8, 77.2), turned to 0 degrees
- moved R8 39.2 mm to (107.0, 106.0), turned to 0 degrees
- moved C16 37.5 mm to (121.0, 77.4), turned to 180 degrees
- moved D3 35.4 mm to (107.0, 103.5), turned to 180 degrees
- moved IC1 35.0 mm to (103.3, 97.7), turned to 90 degrees
- moved Q2 33.8 mm to (128.7, 72.2), turned to 0 degrees
- moved R11 32.8 mm to (173.6, 93.3)
- moved R13 32.4 mm to (124.5, 72.9), turned to 90 degrees
- moved C4 31.7 mm to (137.5, 57.0), turned to 0 degrees
- moved U2 29.8 mm to (166.6, 93.1), turned to 90 degrees
- moved R1 29.3 mm to (146.2, 60.7), turned to 90 degrees
- moved C13 28.1 mm to (108.3, 99.5), turned to 90 degrees
- moved SW1 26.6 mm to (139.8, 60.7), turned to 180 degrees
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Routing:
- net /DIG_0: track 0.00 -> 110.4 mm, vias 0 -> 1
- net /SEG_D: track 0.00 -> 94.0 mm, vias 0 -> 3
- net /DIG_1: track 0.00 -> 88.6 mm, vias 0 -> 1
- net /SEG_G: track 0.00 -> 86.7 mm, vias 0 -> 3
- net /SEG_F: track 0.00 -> 79.3 mm, vias 0 -> 3
- net /SEG_C: track 0.00 -> 74.8 mm, vias 0 -> 4
- net /DIG_2: track 0.00 -> 69.1 mm, vias 0 -> 1
- net /SEG_E: track 0.00 -> 69.0 mm
- net /SEG_B: track 0.00 -> 59.9 mm
- net /SEG_DP: track 0.00 -> 59.6 mm
- net /SEG_A: track 0.00 -> 58.8 mm, vias 0 -> 1
- net /DIG_3: track 0.00 -> 47.6 mm, vias 0 -> 1
- net +3V3: track 0.00 -> 16.6 mm, vias 0 -> 2
- net Net-(D4-A): track 0.00 -> 14.7 mm
- net +5V: track 0.00 -> 13.8 mm
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