File: PCB_V01/MOUNTAIN_IN_THE_POCKET/MOUNTAIN_IN_THE_POCKET.kicad_pcb (KiCad board)
At the start: 2 copper layers, 61 parts, among them IC1 AZ1117CH-3.3TRG1, J1 CON_ALIM, Q2 2N7002, SW1 SW_MEC_5E, SW2 SW_MEC_5E, U1 AP63205WU, U2 AS1115-BSST

Commit message: actualizado routing
Parts:
- moved C13 2.89 mm to (107.6, 96.7)
- moved C15 2.89 mm to (100.8, 100.7)
- moved D3 2.89 mm to (106.3, 100.8)
- moved IC1 2.89 mm to (102.6, 94.9)
- moved R8 2.89 mm to (106.3, 103.2)
- moved R11 0.84 mm to (174.4, 93.0)
- moved D5 0.84 mm to (159.9, 34.3)
- moved D6 0.84 mm to (159.9, 61.9)
- moved D7 0.84 mm to (159.9, 48.1)
- moved D8 0.84 mm to (159.9, 75.7)
- moved U2 0.84 mm to (167.4, 92.8)
- moved C14 0.81 mm to (161.8, 90.3)

Commit message: actu routing
Parts:
- removed VR1: 3362P-1-103LF, 3362P-1-103LF-pretty:3362P_1
- added H1: MountingHole, MountingHole:MountingHole_3.2mm_M3, F.Cu at (191.6, 102.6)
- added H2: MountingHole, MountingHole:MountingHole_3.2mm_M3, F.Cu at (191.4, 31.4)
- added H3: MountingHole, MountingHole:MountingHole_3.2mm_M3, F.Cu at (50.6, 31.2)
- added H4: MountingHole, MountingHole:MountingHole_3.2mm_M3, F.Cu at (50.4, 102.8)
- added TP1: TEST_VBUS, TestPoint:TestPoint_THTPad_D1.0mm_Drill0.5mm, F.Cu at (204.2, 70.6)
- added TP2: TEST_VCC, TestPoint:TestPoint_THTPad_D1.0mm_Drill0.5mm, F.Cu at (209.8, 64.6)
- added TP3: TEST_5V, TestPoint:TestPoint_THTPad_D1.0mm_Drill0.5mm, F.Cu at (207.8, 78.0)
- added TP4: TEST_3V3, TestPoint:TestPoint_THTPad_D1.0mm_Drill0.5mm, F.Cu at (221.4, 64.6)
- added TP5: TEST_GND, TestPoint:TestPoint_THTPad_D1.0mm_Drill0.5mm, F.Cu at (216.2, 82.8)
- added TP6: TEST_SDA, TestPoint:TestPoint_THTPad_D1.0mm_Drill0.5mm, F.Cu at (227.2, 70.4)
- added TP7: TEST_SCL, TestPoint:TestPoint_THTPad_D1.0mm_Drill0.5mm, F.Cu at (224.4, 78.0)
- R2: footprint LIB_HUELLAS_MITP:NORPS12 -> OptoDevice:R_LDR_5.1x4.3mm_P3.4mm_Vertical
- moved D5 63.9 mm to (162.3, 98.1), turned to 180 degrees
- moved R11 58.3 mm to (148.6, 40.8), turned to -90 degrees
- moved U2 54.8 mm to (154.8, 39.6), turned to -90 degrees
- moved C14 48.3 mm to (160.4, 42.1), turned to -90 degrees
- moved S1 43.8 mm to (131.0, 40.6), turned to 90 degrees
- moved C2 38.8 mm to (123.0, 44.8), turned to 0 degrees
- moved D7 36.3 mm to (162.3, 84.3), turned to 180 degrees
- moved R15 34.8 mm to (105.0, 17.6)
- moved R2 30.7 mm to (108.3, 22.4), turned to 180 degrees
- moved C1 25.6 mm to (109.4, 18.8), turned to 180 degrees
- moved R8 24.6 mm to (101.8, 79.0), turned to 180 degrees
- moved C15 20.1 mm to (107.3, 81.7), turned to 0 degrees
- moved D3 19.7 mm to (101.8, 81.5), turned to 0 degrees
- moved D8 19.1 mm to (162.3, 56.7), turned to 180 degrees
- moved C5 17.3 mm to (121.9, 58.8)
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Connections:
- R15 pad 2: Net-(VR1-CW) -> /PIN_LDR
- R2 pad 2: Net-(VR1-CCW) -> /PIN_LDR
- S2 pad 2: /SCL -> /SDA
- S2 pad 3: /SDA -> /SCL
- UC1 pad 1: unconnected-(UC1-3V3-Pad1) -> +3V3
- UC1 pad 15: /PIN_BUZZER -> unconnected-(UC1-GPIO13-Pad15)
- UC1 pad 21: unconnected-(UC1-GPIO23-Pad21) -> /PIN_SEN0137
- UC1 pad 27: unconnected-(UC1-GPIO19-Pad27) -> /PIN_BUTTON_1
- UC1 pad 28: unconnected-(UC1-GPIO18-Pad28) -> /PIN_BUTTON_2
- UC1 pad 30: /PIN_BUTTON_1 -> /PIN_BUZZER
- UC1 pad 31: /PIN_BUTTON_2 -> unconnected-(UC1-GPIO16-Pad31)
- UC1 pad 32: /PIN_SEN0137 -> unconnected-(UC1-GPIO04-Pad32)
Routing:
- net +3V3: track 16.4 -> 63.0 mm, vias 2 -> 0
- net /DIG_0: track 110.4 -> 88.9 mm
- net /DIG_3: track 48.1 -> 65.1 mm
- net /SDA: track 5.38 -> 21.4 mm
- net /PIN_LDR: track 0.00 -> 14.0 mm
- net /PIN_BUZZER: track 0.00 -> 10.2 mm
- net /PIN_BUTTON_2: track 5.53 -> 14.8 mm
- net /PIN_BUTTON_1: track 5.38 -> 14.1 mm
- net /SCL: track 13.2 -> 21.7 mm
- net /DIG_1: track 88.6 -> 81.2 mm
- net /DIG_2: track 69.1 -> 73.0 mm
- net /SEG_D: track 94.0 -> 91.6 mm
- net Net-(U2-ISET): track 4.64 -> 2.91 mm
- net /SEG_A: track 58.8 -> 57.2 mm
- net Net-(D4-A): track 14.7 -> 15.4 mm
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Other:
- board outline added: 154.8 x 84.8 mm
- board text added: "S1"
